Commit message: 切换了带有夹爪的urdf

File: install/dummy-ros2_description/share/dummy-ros2_description/urdf/dummy-ros2-gazebo.xacro (robot description, xacro)
@@ -123,5 +123,5 @@
   </inertial>
   <visual>
-    <origin xyz="0.0346 0.234017 -0.318" rpy="0 0 0"/>
+    <origin xyz="-0.01 -0.08 -0.318" rpy="0 0 0"/>
     <geometry>
       <mesh filename="file://$(find dummy-ros2_description)/meshes/link5_1_1.stl" scale="0.001 0.001 0.001"/>
@@ -130,5 +130,5 @@
   </visual>
   <collision>
-    <origin xyz="0.0346 0.234017 -0.318" rpy="0 0 0"/>
+    <origin xyz="-0.01 -0.08 -0.318" rpy="0 0 0"/>
     <geometry>
       <mesh filename="file://$(find dummy-ros2_description)/meshes/link5_1_1.stl" scale="0.001 0.001 0.001"/>
@@ -144,5 +144,5 @@
   </inertial>
   <visual>
-    <origin xyz="0.016 0.290517 -0.318" rpy="0 0 0"/>
+    <origin xyz="0.013 0.2465 -0.3545" rpy="0 0 3.141592654"/>
     <geometry>
       <mesh filename="file://$(find dummy-ros2_description)/meshes/link6_1_1.stl" scale="0.001 0.001 0.001"/>
@@ -151,5 +151,5 @@
   </visual>
   <collision>
-    <origin xyz="0.016 0.290517 -0.318" rpy="0 0 0"/>
+    <origin xyz="0.013 0.2465 -0.3545" rpy="0 0 0"/>
     <geometry>
       <mesh filename="file://$(find dummy-ros2_description)/meshes/link6_1_1.stl" scale="0.001 0.001 0.001"/>
@@ -297,5 +297,5 @@
 <!-- D435深度相机安装在J6末端 -->
 <xacro:sensor_d435 parent="link6_1_1" name="d435" use_nominal_extrinsics="true">
-  <origin xyz="0.00 0.006 0.02" rpy="0 0 -1.5708"/>
+  <origin xyz="0.00 -0.04 0.03" rpy="0 0 -1.5708"/>
 </xacro:sensor_d435>
 <!-- Gazebo D435相机插件 -->

File: install/dummy-ros2_description/share/dummy-ros2_description/urdf/dummy-ros2.xacro (robot description, xacro)
@@ -116,5 +116,5 @@
   </inertial>
   <visual>
-    <origin xyz="0.0346 0.234017 -0.318" rpy="0 0 0"/>
+    <origin xyz="-0.01 -0.08 -0.318" rpy="0 0 0"/>
     <geometry>
       <mesh filename="file://$(find dummy-ros2_description)/meshes/link5_1_1.stl" scale="0.001 0.001 0.001"/>
@@ -123,5 +123,5 @@
   </visual>
   <collision>
-    <origin xyz="0.0346 0.234017 -0.318" rpy="0 0 0"/>
+    <origin xyz="-0.01 -0.08 -0.318" rpy="0 0 0"/>
     <geometry>
       <mesh filename="file://$(find dummy-ros2_description)/meshes/link5_1_1.stl" scale="0.001 0.001 0.001"/>
@@ -136,5 +136,5 @@
   </inertial>
   <visual>
-    <origin xyz="0.016 0.290517 -0.318" rpy="0 0 0"/>
+    <origin xyz="0.013 0.2465 -0.3545" rpy="0 0 3.141592654"/>
     <geometry>
       <mesh filename="file://$(find dummy-ros2_description)/meshes/link6_1_1.stl" scale="0.001 0.001 0.001"/>
@@ -143,5 +143,5 @@
   </visual>
   <collision>
-    <origin xyz="0.016 0.290517 -0.318" rpy="0 0 0"/>
+    <origin xyz="0.013 0.2465 -0.3545" rpy="0 0 0"/>
     <geometry>
       <mesh filename="file://$(find dummy-ros2_description)/meshes/link6_1_1.stl" scale="0.001 0.001 0.001"/>

Commit message: 更新了urdf参数的准确度

File: install/dummy-ros2_description/share/dummy-ros2_description/urdf/dummy-ros2-gazebo.xacro (robot description, xacro)
@@ -8,5 +8,5 @@
   <parent link="world" />
   <child link="base_link" />
-  <origin xyz="0.0 0.0 0.0" rpy="0.0 0.0 0.0" />
+  <origin xyz="0.0 0.0 0.0" rpy="3.1415926536 3.1415926536 0.0" />
 </joint>
 <!-- 基座链接 -->
@@ -170,5 +170,5 @@
   <parent link="link1_1_1"/>
   <child link="link2_1_1"/>
-  <axis xyz="1.0 0.0 0.0"/>
+  <axis xyz="1.0 0.0 -0.0"/>
   <limit lower="-1.308997" upper="1.570796" effort="150" velocity="3.15"/>
   <dynamics damping="10.0" friction="1.0"/>
@@ -178,5 +178,5 @@
   <parent link="link2_1_1"/>
   <child link="link3_1_1"/>
-  <axis xyz="1.0 0.0 0.0"/>
+  <axis xyz="1.0 -0.0 -0.0"/>
   <limit lower="-1.570796" upper="1.570796" effort="150" velocity="3.15"/>
   <dynamics damping="10.0" friction="1.0"/>
@@ -194,13 +194,13 @@
   <parent link="link4_1_1"/>
   <child link="link5_1_1"/>
-  <axis xyz="-1.0 0.0 0.0"/>
+  <axis xyz="-1.0 -0.0 0.0"/>
   <limit lower="-1.570796" upper="1.570796" effort="150" velocity="3.15"/>
   <dynamics damping="10.0" friction="1.0"/>
 </joint>
 <joint name="joint6" type="revolute">
-  <origin xyz="0.0186 -0.0565 0.0" rpy="0 0 0"/>
+  <origin xyz="0.0186 -0.0605 0.0" rpy="0 0 0"/>
   <parent link="link5_1_1"/>
   <child link="link6_1_1"/>
-  <axis xyz="0.0 1.0 0.0"/>
+  <axis xyz="0.0 1.0 -0.0"/>
   <limit lower="-3.14" upper="3.14" effort="150" velocity="3.15"/>
   <dynamics damping="10.0" friction="1.0"/>

File: install/dummy-ros2_description/share/dummy-ros2_description/urdf/dummy-ros2.xacro (robot description, xacro)
@@ -205,5 +205,5 @@
 </joint>
 <joint name="joint6" type="revolute">
-  <origin xyz="0.0186 -0.0565 0.0" rpy="0 0 0"/>
+  <origin xyz="0.0186 -0.0605 0.0" rpy="0 0 0"/>
   <parent link="link5_1_1"/>
   <child link="link6_1_1"/>
