Commit message: 整体版本调整

File: install/dummy-ros2_description/share/dummy-ros2_description/urdf/dummy-ros2.xacro (robot description, xacro)
@@ -143,7 +143,48 @@
   </visual>
   <collision>
-    <origin xyz="0.013 0.2465 -0.3545" rpy="0 0 0"/>
+    <origin xyz="0.013 0.2465 -0.3545" rpy="0 0 3.141592654"/>
     <geometry>
       <mesh filename="file://$(find dummy-ros2_description)/meshes/link6_1_1.stl" scale="0.001 0.001 0.001"/>
+    </geometry>
+  </collision>
+</link>
+<!-- 夹爪链接 -->
+<link name="gripper_left_link">
+  <inertial>
+    <origin xyz="0 0 0" rpy="0 0 0"/>
+    <mass value="0.05"/>
+    <inertia ixx="1e-5" iyy="1e-5" izz="1e-5" ixy="0" iyz="0" ixz="0"/>
+  </inertial>
+  <visual>
+    <origin xyz="0 0 0" rpy="0 0 0"/>
+    <geometry>
+      <mesh filename="file://$(find dummy-ros2_description)/meshes/gripper.stl" scale="0.001 0.001 0.001"/>
+    </geometry>
+    <material name="silver"/>
+  </visual>
+  <collision>
+    <origin xyz="0 0 0" rpy="0 0 0"/>
+    <geometry>
+      <mesh filename="file://$(find dummy-ros2_description)/meshes/gripper.stl" scale="0.001 0.001 0.001"/>
+    </geometry>
+  </collision>
+</link>
+<link name="gripper_right_link">
+  <inertial>
+    <origin xyz="0 0 0" rpy="0 0 0"/>
+    <mass value="0.05"/>
+    <inertia ixx="1e-5" iyy="1e-5" izz="1e-5" ixy="0" iyz="0" ixz="0"/>
+  </inertial>
+  <visual>
+    <origin xyz="0 0 0" rpy="0 0 0"/>
+    <geometry>
+      <mesh filename="file://$(find dummy-ros2_description)/meshes/gripper.stl" scale="0.001 0.001 0.001"/>
+    </geometry>
+    <material name="silver"/>
+  </visual>
+  <collision>
+    <origin xyz="0 0 0" rpy="0 0 0"/>
+    <geometry>
+      <mesh filename="file://$(find dummy-ros2_description)/meshes/gripper.stl" scale="0.001 0.001 0.001"/>
     </geometry>
   </collision>
@@ -155,6 +196,6 @@
   <axis xyz="0.0 0.0 1.0"/>
   <limit
-    lower="-3.141593"
-    upper="3.141593"
+    lower="-2.967059728"
+    upper="2.967059"
     effort="150"
     velocity="3.15"/>
@@ -215,3 +256,26 @@
     velocity="3.15" />
 </joint>
+<!-- 夹爪关节 -->
+<joint name="joint7" type="prismatic">
+  <origin xyz="-0.011000 0.232000 0.353000" rpy="3.141592654 0.000000 0.000000"/>
+  <parent link="link6_1_1"/>
+  <child link="gripper_left_link"/>
+  <axis xyz="1.0 0.0 0.0"/>
+  <limit
+    lower="0.000000"
+    upper="0.025000"
+    effort="50"
+    velocity="0.5"/>
+</joint>
+<joint name="joint8" type="prismatic">
+  <origin xyz="0.011000 0.232000 -0.354500" rpy="0.000000 0.000000 3.141590"/>
+  <parent link="link6_1_1"/>
+  <child link="gripper_right_link"/>
+  <axis xyz="-1.0 0.0 0.0"/>
+  <limit
+    lower="-0.025000"
+    upper="0.000000"
+    effort="50"
+    velocity="0.5"/>
+</joint>
 </robot>

File: install/dummy_moveit_config/share/dummy_moveit_config/config/dummy-ros2.ros2_control.xacro (robot description, xacro)
@@ -69,4 +69,25 @@
                 <state_interface name="velocity"/>
             </joint>
+            <!-- 夹爪关节配置 -->
+            <joint name="joint7">
+                <command_interface name="position">
+                    <param name="min">0.0</param>
+                    <param name="max">0.04</param>
+                </command_interface>
+                <state_interface name="position">
+                    <param name="initial_value">${initial_positions['joint7']}</param>
+                </state_interface>
+                <state_interface name="velocity"/>
+            </joint>
+            <joint name="joint8">
+                <command_interface name="position">
+                    <param name="min">-0.04</param>
+                    <param name="max">0.0</param>
+                </command_interface>
+                <state_interface name="position">
+                    <param name="initial_value">${initial_positions['joint8']}</param>
+                </state_interface>
+                <state_interface name="velocity"/>
+            </joint>
         </ros2_control>
     </xacro:macro>
